Commit message: feat: add field acceptance extrinsics

File: urdf/tracked_chassis.urdf.xacro (robot description, xacro)
@@ -3,6 +3,7 @@
   <xacro:arg
     name="calibration_file"
-    default="$(find tracked_chassis_description)/config/cad_alignment.initial_guess.yaml"/>
-  <xacro:property name="calib" value="${xacro.load_yaml(calibration_file)}"/>
+    default="$(find tracked_chassis_description)/config/field_acceptance.yaml"/>
+  <xacro:property name="calibration_file_path" value="$(arg calibration_file)"/>
+  <xacro:property name="calib" value="${xacro.load_yaml(calibration_file_path)}"/>
   <xacro:property name="base_link_z" value="${calib['base_link_z']}"/>
   <xacro:property name="base_to_cad" value="${calib['base_link_to_cad']}"/>

File: urdf/tracked_chassis_runtime.urdf.xacro (robot description, xacro)
@@ -3,6 +3,7 @@
   <xacro:arg
     name="calibration_file"
-    default="$(find tracked_chassis_description)/config/cad_alignment.initial_guess.yaml"/>
-  <xacro:property name="calib" value="${xacro.load_yaml(calibration_file)}"/>
+    default="$(find tracked_chassis_description)/config/field_acceptance.yaml"/>
+  <xacro:property name="calibration_file_path" value="$(arg calibration_file)"/>
+  <xacro:property name="calib" value="${xacro.load_yaml(calibration_file_path)}"/>
   <xacro:property name="base_link_z" value="${calib['base_link_z']}"/>
   <xacro:property name="base_to_cad" value="${calib['base_link_to_cad']}"/>
